File: schematic/board.sch (EAGLE design)
At the start: 22 parts, among them U1 STM32F103C8T6

Commit message: Прикидки размеров платы
Parts:
- removed U$5: E01-ML01DP5, ebyte-radio:E01-ML01DP5
- removed U$7: CST2-JTAG2X5-1.27MM-R, IDC:CST2-JTAG2X5-1.27MM-R
- added J1: (no value), SparkFun-Connectors:CONN_04X2
- added P1: S8B-PH-K, con-jst-ph:S8B-PH-K
- U$2: value CST2-JTAG -> TFP09-2-12B; device IDC:CST2-JTAG -> sdcard:TFP09-2-12B
Connections:
- net +3V3: no longer U$2.3.3V
- net +5V: no longer U$2.5V
- net GND: no longer U$2.GND
- net JTCK: no longer U$2.TCLK
- net JTDI: no longer U$2.TDI
- net JTDO: no longer U$2.TDO
- net JTMS: no longer U$2.TMS
- net NRST: no longer U$2.NRST
Changed lines of the file:
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@@
 <part name="GND5" library="supply1" library_urn="urn:adsk.eagle:library:371" deviceset="GND" device=""/>
 <part name="GND6" library="supply1" library_urn="urn:adsk.eagle:library:371" deviceset="GND" device=""/>
-<part name="U$2" library="IDC" deviceset="CST2-JTAG" device=""/>
 <part name="U2" library="SparkFun-IC-Power" deviceset="V_REG_LM1117" device="SOT223"/>
 <part name="Y1" library="SparkFun-Clocks" deviceset="CRYSTAL" device="PTH-HC49US"/>
@@
 <part name="R2" library="SparkFun-Resistors" deviceset="RESISTOR" device="0603" value=" "/>
 <part name="U$4" library="ebyte-radio" deviceset="E01-ML01SP4" device=""/>
-<part name="U$5" library="ebyte-radio" deviceset="E01-ML01DP5" device=""/>
 <part name="U$6" library="IDC" deviceset="DS-1013-20" device="LOCK"/>
-<part name="U$7" library="IDC" deviceset="CST2-JTAG" device="2X5-1.27MM-R"/>
+<part name="J1" library="SparkFun-Connectors" deviceset="CONN_04X2" device=""/>
+<part name="U$2" library="sdcard" deviceset="TFP09-2-12B" device=""/>
+<part name="P1" library="con-jst-ph" deviceset="S8B-PH-K" device=""/>
 </parts>
 <sheets>
@@
 <attribute name="VALUE" x="-172.72" y="-50.8" size="1.778" layer="96" rot="MR0"/>
 </instance>
-<instance part="U$2" gate="G$1" x="-160.02" y="167.64" smashed="yes">
-<attribute name="VALUE" x="-171.45" y="157.734" size="1.778" layer="96" font="vector"/>
-<attribute name="NAME" x="-171.45" y="175.768" size="1.778" layer="95" font="vector"/>
-</instance>
 <instance part="U2" gate="G$1" x="-160.02" y="236.22" smashed="yes">
 <attribute name="NAME" x="-157.48" y="228.6" size="1.778" layer="95"/>
@@
 <attribute name="VALUE" x="53.34" y="-43.18" size="1.27" layer="96"/>
 </instance>
-<instance part="U$5" gate="G$1" x="132.08" y="-30.48" smashed="yes">
-<attribute name="NAME" x="124.46" y="-17.78" size="1.27" layer="95"/>
-<attribute name="VALUE" x="124.46" y="-43.18" size="1.27" layer="96"/>
-</instance>
 <instance part="U$6" gate="G$1" x="-73.66" y="78.74" smashed="yes">
 <attribute name="VALUE" x="-77.47" y="61.214" size="1.778" layer="96" font="vector"/>
 <attribute name="NAME" x="-77.47" y="91.948" size="1.778" layer="95" font="vector"/>
 </instance>
-<instance part="U$7" gate="G$1" x="-63.5" y="149.86" smashed="yes">
-<attribute name="VALUE" x="-74.93" y="139.954" size="1.778" layer="96" font="vector"/>
-<attribute name="NAME" x="-74.93" y="157.988" size="1.778" layer="95" font="vector"/>
+<instance part="J1" gate="G$1" x="2.54" y="-30.48" smashed="yes">
+<attribute name="VALUE" x="-1.27" y="-37.846" size="1.778" layer="96" font="vector"/>
+<attribute name="NAME" x="-1.524" y="-22.352" size="1.778" layer="95" font="vector"/>
+</instance>
+<instance part="U$2" gate="G$1" x="-35.56" y="-88.9" smashed="yes">
+<attribute name="NAME" x="-48.26" y="-66.04" size="1.27" layer="95" rot="MR0"/>
+<attribute name="VALUE" x="-50.8" y="-114.3" size="1.27" layer="96"/>
+</instance>
+<instance part="P1" gate="G$1" x="-17.78" y="-30.48" smashed="yes">
+<attribute name="NAME" x="-19.05" y="-17.145" size="1.778" layer="95"/>
+<attribute name="VALUE" x="-19.05" y="-43.18" size="1.778" layer="95"/>
 </instance>
 </instances>
@@
 <wire x1="-182.88" y1="160.02" x2="-182.88" y2="162.56" width="0.1524" layer="91"/>
 <wire x1="-182.88" y1="162.56" x2="-175.26" y2="162.56" width="0.1524" layer="91"/>
-<pinref part="U$2" gate="G$1" pin="GND"/>
 </segment>
 <segment>
@@
 <wire x1="-111.76" y1="172.72" x2="-144.78" y2="172.72" width="0.1524" layer="91"/>
 <label x="-144.78" y="172.72" size="1.778" layer="95"/>
-<pinref part="U$2" gate="G$1" pin="TMS"/>
 </segment>
 <segment>
@@
 <wire x1="-111.76" y1="170.18" x2="-144.78" y2="170.18" width="0.1524" layer="91"/>
 <label x="-144.78" y="170.18" size="1.778" layer="95"/>
-<pinref part="U$2" gate="G$1" pin="TCLK"/>
 </segment>
 <segment>
@@
 <wire x1="-111.76" y1="167.64" x2="-144.78" y2="167.64" width="0.1524" layer="91"/>
 <label x="-144.78" y="167.64" size="1.778" layer="95"/>
-<pinref part="U$2" gate="G$1" pin="TDO"/>
 </segment>
 <segment>
@@
 <wire x1="-111.76" y1="165.1" x2="-144.78" y2="165.1" width="0.1524" layer="91"/>
 <label x="-144.78" y="165.1" size="1.778" layer="95"/>
-<pinref part="U$2" gate="G$1" pin="TDI"/>
 </segment>
 <segment>
@@
 <segment>
 <wire x1="-144.78" y1="162.56" x2="-132.08" y2="162.56" width="0.1524" layer="91"/>
-<pinref part="U$2" gate="G$1" pin="NRST"/>
 <label x="-144.78" y="162.56" size="1.778" layer="95"/>
 </segment>
@@
 <wire x1="-182.88" y1="180.34" x2="-182.88" y2="172.72" width="0.1524" layer="91"/>
 <wire x1="-182.88" y1="172.72" x2="-175.26" y2="172.72" width="0.1524" layer="91"/>
-<pinref part="U$2" gate="G$1" pin="3.3V"/>
 </segment>
 <segment>
@@
 <wire x1="-187.96" y1="177.8" x2="-187.96" y2="170.18" width="0.1524" layer="91"/>
 <wire x1="-187.96" y1="170.18" x2="-175.26" y2="170.18" width="0.1524" layer="91"/>
-<pinref part="U$2" gate="G$1" pin="5V"/>
-</segment>
-<segment>
+</segment>
+<segment>

Commit message: Замороженное состояние
Parts:
- removed U$6: DS-1013-20LOCK, IDC:DS-1013-20LOCK
- added U3: LSM6DS3, LSM6DS3:LSM6DS3
- added U4: LSM303CTR, LSM303CTR:LSM303CTR
Changed lines of the file:
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@@
 <part name="R2" library="SparkFun-Resistors" deviceset="RESISTOR" device="0603" value=" "/>
 <part name="U$4" library="ebyte-radio" deviceset="E01-ML01SP4" device=""/>
-<part name="U$6" library="IDC" deviceset="DS-1013-20" device="LOCK"/>
 <part name="J1" library="SparkFun-Connectors" deviceset="CONN_04X2" device=""/>
 <part name="U$2" library="sdcard" deviceset="TFP09-2-12B" device=""/>
 <part name="P1" library="con-jst-ph" deviceset="S8B-PH-K" device=""/>
+<part name="U3" library="LSM6DS3" deviceset="LSM6DS3" device=""/>
+<part name="U4" library="LSM303CTR" deviceset="LSM303CTR" device=""/>
 </parts>
 <sheets>
@@
 <attribute name="VALUE" x="53.34" y="-43.18" size="1.27" layer="96"/>
 </instance>
-<instance part="U$6" gate="G$1" x="-73.66" y="78.74" smashed="yes">
-<attribute name="VALUE" x="-77.47" y="61.214" size="1.778" layer="96" font="vector"/>
-<attribute name="NAME" x="-77.47" y="91.948" size="1.778" layer="95" font="vector"/>
-</instance>
 <instance part="J1" gate="G$1" x="2.54" y="-30.48" smashed="yes">
 <attribute name="VALUE" x="-1.27" y="-37.846" size="1.778" layer="96" font="vector"/>
@@
 <attribute name="VALUE" x="-19.05" y="-43.18" size="1.778" layer="95"/>
 </instance>
+<instance part="U3" gate="G$1" x="-58.42" y="66.04" smashed="yes">
+<attribute name="NAME" x="-71.1404" y="79.2692" size="1.78085" layer="95"/>
+<attribute name="VALUE" x="-71.1211" y="50.7986" size="1.778159375" layer="96"/>
+</instance>
+<instance part="U4" gate="G$1" x="-60.96" y="106.68" smashed="yes">
+<attribute name="NAME" x="-71.145" y="119.8951" size="1.78238125" layer="95"/>
+<attribute name="VALUE" x="-71.1274" y="91.6577" size="1.779290625" layer="96"/>
+</instance>
 </instances>
